Commit message: ik works, code has to be rewritten

File: script/delta_robot_description/urdf/delta_robot.urdf (robot description, URDF)
Before this commit: robot delta_robot, 7 links, 6 joints
Joints:
- joint rod_1_end-effector_joint: origin xyz=450 0 0 -> xyz=0 0 -450
- joint rod_1_joint: origin xyz=0. 0. 0. rpy=0 0.7853981634 0 -> xyz=0. 0. 0. rpy=0 0 0
- joint rod_2_end-effector_joint: origin xyz=450 0 0 -> xyz=0 0 -450
- joint rod_2_joint: origin xyz=0 0 0 rpy=0 2.35619449 0 -> xyz=0 0 0 rpy=0 0 0

File: script/delta_robot_description/urdf/delta_robot_1.urdf (robot description, URDF)
Before this commit: robot delta_robot, 4 links, 3 joints
Joints:
- joint rod_1_end-effector_joint: origin xyz=450 0 0 -> xyz=0 0 -450

File: script/delta_robot_description/urdf/delta_robot_2.urdf (robot description, URDF)
Before this commit: robot delta_robot, 4 links, 3 joints
Joints:
- joint carriage_2_joint: axis -1 0 -1 -> 1 0 1
- joint rod_2_end-effector_joint: origin xyz=450 0 0 -> xyz=0 0 -450

Commit message: added link

File: script/delta_robot_description/urdf/delta_robot.urdf (robot description, URDF)
Before this commit: robot delta_robot, 7 links, 6 joints
Links:
- added link rod_3_end-effector_link; visual mesh filename=../meshes/end-effector_joint.stl
- added link rod_3_link; visual mesh filename=../meshes/link_1.stl
Joints:
- added joint rod_3_end-effector_joint: type fixed, parent rod_3_link, child rod_3_end-effector_link, origin xyz=0 0 -450
- added joint rod_3_joint: type revolute, parent carriage_2_link, child rod_3_link, origin xyz=45 0 0 rpy=0 0 0, axis 0 1 0, limit lower=0 upper=6.28 effort=0 velocity=0

Commit message: collision checking has to be fixed

File: script/delta_robot_description/urdf/delta_robot.urdf (robot description, URDF)
Before this commit: robot delta_robot, 9 links, 8 joints
Links:
- removed link rod_1_end-effector_link
- added link end_effector_link; visual mesh filename=../meshes/end_effector.stl
- link rails_link: geometry collision mesh filename=../meshes/rails_collision.stl scale=0.6 1.5 0.6; visual mesh filename=../meshes/rails.stl
- link rod_1_link: geometry collision mesh filename=../meshes/link_1.stl; visual mesh filename=../meshes/link_1.stl
- link rod_2_link: geometry collision mesh filename=../meshes/link_2.stl; visual mesh filename=../meshes/link_2.stl
- link rod_3_link: geometry visual mesh filename=../meshes/link_1_c2.stl
Joints:
- joint rod_1_end-effector_joint: axis (none) -> 0 1 0; child rod_1_end-effector_link -> end_effector_link; limit (none) -> lower=0 upper=6.28 effort=0 velocity=0; type fixed -> revolute

Commit message: added collision

File: script/delta_robot_description/urdf/delta_robot.urdf (robot description, URDF)
Before this commit: robot delta_robot, 9 links, 8 joints
Links:
- link rails_link: geometry collision mesh filename=../meshes/rails_collision.stl scale=0.9 1.5 0.9; visual mesh filename=../meshes/rails.stl
