Commit message: added robot description

File: src/deltarobot_description/urdf/delta_robot.urdf (robot description, URDF)
Before this commit: robot delta_robot, 9 links, 8 joints
Links:
- link carriage_1_link: geometry visual mesh filename=package://deltarobot_description/meshes/carriage_1.stl
- link carriage_2_link: geometry visual mesh filename=package://deltarobot_description/meshes/carriage_2.stl
- link end_effector_link: geometry visual mesh filename=package://deltarobot_description/meshes/end_effector.stl
- link rails_link: geometry collision mesh filename=package://deltarobot_description/meshes/carriage_1.stl scale=0.9 1.5 0.9; visual mesh filename=package://deltarobot_description/meshes/rails.stl
- link rod_1_link: geometry collision mesh filename=package://deltarobot_description/meshes/link_1.stl; visual mesh filename=package://deltarobot_description/meshes/link_1.stl
- link rod_2_end-effector_link: geometry visual mesh filename=package://deltarobot_description/meshes/end-effector_joint.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
- link rod_2_link: geometry collision mesh filename=package://deltarobot_description/meshes/link_2.stl; visual mesh filename=package://deltarobot_description/meshes/link_2.stl
- link rod_3_end-effector_link: geometry visual mesh filename=package://deltarobot_description/meshes/end-effector_joint.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
- link rod_3_link: geometry visual mesh filename=package://deltarobot_description/meshes/link_1_c2.stl

Commit message: .

File: src/deltarobot_description/urdf/delta_robot.urdf (robot description, URDF)
Before this commit: robot delta_robot, 9 links, 8 joints
Links:
- link rails_link: geometry collision mesh filename=package://deltarobot_description/meshes/rails_collision.stl scale=0.9 1.5 0.9; visual mesh filename=package://deltarobot_description/meshes/rails.stl
