Commit message: added urdf reduced

File: src/deltarobot_description/urdf/deltarobot_chain_1_reduced.urdf (robot description, URDF)
Before this commit: robot delta_robot, 4 links, 3 joints
Links:
- link rails_link: geometry collision mesh filename=/home/ostifede02/Documents/2dr_ws/src/deltarobot_descriptio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 scale=0.9 1.5 0.9
- link rod_1_link: geometry collision mesh filename=/home/ostifede02/Documents/2dr_ws/src/deltarobot_descriptio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

File: src/deltarobot_description/urdf/deltarobot_chain_2_reduced.urdf (robot description, URDF)
Before this commit: robot delta_robot, 9 links, 8 joints
Links:
- removed link carriage_1_link
- removed link end_effector_link
- removed link rod_1_link
- removed link rod_2_end-effector_link
- removed link rod_3_end-effector_link
- removed link rod_3_link
- added link rod_2_end_effector_link
- link carriage_2_link: geometry 
- link rails_link: geometry collision mesh filename=/home/ostifede02/Documents/2dr_ws/src/deltarobot_descriptio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 scale=0.9 1.5 0.9
- link rod_2_link: geometry collision mesh filename=/home/ostifede02/Documents/2dr_ws/src/deltarobot_descriptio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
Joints:
- removed joint carriage_1_joint
- removed joint rod_1_end-effector_joint
- removed joint rod_1_joint
- removed joint rod_2_end-effector_joint
- removed joint rod_3_end-effector_joint
- removed joint rod_3_joint
- added joint rod_2_end_effector_joint: type fixed, parent rod_2_link, child rod_2_end_effector_link, origin xyz=0 0 -450
