Commit message: gui control works

File: src/deltarobot_description/urdf/deltarobot.urdf (robot description, URDF)
Before this commit: robot delta_robot, 9 links, 8 joints
Links:
- removed link rod_2_end-effector_link
- removed link rod_3_end-effector_link
- added link rod_2_end_effector_link; visual mesh filename=/home/ostifede02/Documents/2dr_ws/src/deltarobot_descriptio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
- added link rod_3_end_effector_link; visual mesh filename=/home/ostifede02/Documents/2dr_ws/src/deltarobot_descriptio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
- link carriage_1_link: geometry visual mesh filename=/home/ostifede02/Documents/2dr_ws/src/deltarobot_descriptio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
- link carriage_2_link: geometry visual mesh filename=/home/ostifede02/Documents/2dr_ws/src/deltarobot_descriptio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
- link end_effector_link: geometry visual mesh filename=/home/ostifede02/Documents/2dr_ws/src/deltarobot_descriptio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
- link rails_link: geometry collision mesh filename=/home/ostifede02/Documents/2dr_ws/src/deltarobot_descriptio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 scale=0.9 1.5 0.9; visual mesh filename=/home/ostifede02/Documents/2dr_ws/src/deltarobot_descriptio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
- link rod_1_link: geometry collision mesh filename=/home/ostifede02/Documents/2dr_ws/src/deltarobot_descriptio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; visual mesh filename=/home/ostifede02/Documents/2dr_ws/src/deltarobot_descriptio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
- link rod_2_link: geometry collision mesh filename=/home/ostifede02/Documents/2dr_ws/src/deltarobot_descriptio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; visual mesh filename=/home/ostifede02/Documents/2dr_ws/src/deltarobot_descriptio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
- link rod_3_link: geometry visual mesh filename=/home/ostifede02/Documents/2dr_ws/src/deltarobot_descriptio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
Joints:
- removed joint rod_1_end-effector_joint
- removed joint rod_2_end-effector_joint
- removed joint rod_3_end-effector_joint
- added joint rod_1_end_effector_joint: type revolute, parent rod_1_link, child end_effector_link, origin xyz=0 0 -450, axis 0 1 0, limit lower=0 upper=6.28 effort=0 velocity=0
- added joint rod_2_end_effector_joint: type fixed, parent rod_2_link, child rod_2_end_effector_link, origin xyz=0 0 -450
- added joint rod_3_end_effector_joint: type fixed, parent rod_3_link, child rod_3_end_effector_link, origin xyz=0 0 -450

Commit message: three axis work

File: src/deltarobot_description/urdf/deltarobot.urdf (robot description, URDF)
Before this commit: robot delta_robot, 9 links, 8 joints
Links:
- removed link end_effector_link
- removed link rod_1_link
- removed link rod_2_link
- removed link rod_3_link
- added link carriage_3_link; visual mesh filename=carriage.stl
- added link rod_1_end_effector_link
- added link rod_1a_link; collision mesh filename=link.stl; visual mesh filename=link.stl
- added link rod_1a_link_virtual
- added link rod_1b_link; collision mesh filename=link.stl; visual mesh filename=link.stl
- added link rod_1b_link_virtual
- added link rod_2a_link; collision mesh filename=link.stl; visual mesh filename=link.stl
- added link rod_2a_link_virtual
- added link rod_2b_link; collision mesh filename=link.stl; visual mesh filename=link.stl
- added link rod_2b_link_virtual
- added link rod_3a_link; collision mesh filename=link.stl; visual mesh filename=link.stl
- added link rod_3a_link_virtual
- added link rod_3b_link; collision mesh filename=link.stl; visual mesh filename=link.stl
- added link rod_3b_link_virtual
- link carriage_1_link: geometry visual mesh filename=carriage.stl
- link carriage_2_link: geometry visual mesh filename=carriage.stl
- link rails_link: geometry collision mesh filename=rails.stl; visual mesh filename=rails.stl
- link rod_2_end_effector_link: geometry 
- link rod_3_end_effector_link: geometry 
Joints:
- removed joint rod_1_joint
- removed joint rod_2_joint
- removed joint rod_3_joint
- added joint carriage_3_joint: type prismatic, parent rails_link, child carriage_3_link, origin xyz=0. 0. 0. rpy=0 0 0, axis 0.61237244 -0.35355339 0.70710678, limit lower=0 upper=0 effort=0 velocity=0
- added joint rod_1a_x_joint: type revolute, parent carriage_1_link, child rod_1a_link_virtual, origin xyz=25 0. 0. rpy=0 0 0, axis 1 0 0, limit lower=0 upper=0 effort=0 velocity=0
- added joint rod_1a_y_joint: type revolute, parent rod_1a_link_virtual, child rod_1a_link, origin xyz=0. 0. 0. rpy=0 0 0, axis 0 1 0, limit lower=0 upper=0 effort=0 velocity=0
- added joint rod_1b_x_joint: type revolute, parent carriage_1_link, child rod_1b_link_virtual, origin xyz=-25 0. 0. rpy=0 0 0, axis 1 0 0, limit lower=0 upper=0 effort=0 velocity=0
- added joint rod_1b_y_joint: type revolute, parent rod_1b_link_virtual, child rod_1b_link, origin xyz=0. 0. 0. rpy=0 0 0, axis 0 1 0, limit lower=0 upper=0 effort=0 velocity=0
- added joint rod_2a_x_joint: type revolute, parent carriage_2_link, child rod_2a_link_virtual, origin xyz=12.5 -21.650635 0 rpy=0 0 0, axis -0.5 0.8660254 0, limit lower=0 upper=0 effort=0 velocity=0
- added joint rod_2a_y_joint: type revolute, parent rod_2a_link_virtual, child rod_2a_link, origin xyz=0 0 0 rpy=0 0 0, axis -0.8660254 -0.5 0, limit lower=0 upper=0 effort=0 velocity=0
- added joint rod_2b_x_joint: type revolute, parent carriage_2_link, child rod_2b_link_virtual, origin xyz=-12.5 21.650635 0 rpy=0 0 0, axis -0.5 0.8660254 0, limit lower=0 upper=0 effort=0 velocity=0
- added joint rod_2b_y_joint: type revolute, parent rod_2b_link_virtual, child rod_2b_link, origin xyz=0 0 0 rpy=0 0 0, axis -0.8660254 -0.5 0, limit lower=0 upper=0 effort=0 velocity=0
- added joint rod_3a_x_joint: type revolute, parent carriage_3_link, child rod_3a_link_virtual, origin xyz=-12.5 -21.650635 0 rpy=0 0 0, axis -0.5 -0.8660254 0, limit lower=0 upper=0 effort=0 velocity=0
- added joint rod_3a_y_joint: type revolute, parent rod_3a_link_virtual, child rod_3a_link, origin xyz=0 0 0 rpy=0 0 0, axis 0.8660254 -0.5 0, limit lower=0 upper=0 effort=0 velocity=0
- added joint rod_3b_x_joint: type revolute, parent carriage_3_link, child rod_3b_link_virtual, origin xyz=12.5 21.650635 0 rpy=0 0 0, axis -0.5 -0.8660254 0, limit lower=0 upper=0 effort=0 velocity=0
- added joint rod_3b_y_joint: type revolute, parent rod_3b_link_virtual, child rod_3b_link, origin xyz=0 0 0 rpy=0 0 0, axis 0.8660254 -0.5 0, limit lower=0 upper=0 effort=0 velocity=0
- joint carriage_1_joint: axis -1 0 1 -> 0 1 1; limit lower=60 upper=350 effort=0 velocity=0 -> lower=0 upper=0 effort=0 velocity=0
- joint carriage_2_joint: axis 1 0 1 -> -0.61237244 -0.35355339 0.70710678; limit lower=60 upper=350 effort=0 velocity=0 -> lower=0 upper=0 effort=0 velocity=0
- joint rod_1_end_effector_joint: axis 0 1 0 -> (none); child end_effector_link -> rod_1_end_effector_link; limit lower=0 upper=6.28 effort=0 velocity=0 -> (none); origin xyz=0 0 -450 -> xyz=0 0 -400; parent rod_1_link -> rod_1a_link; type revolute -> fixed
- joint rod_2_end_effector_joint: origin xyz=0 0 -450 -> xyz=0 0 -400; parent rod_2_link -> rod_2a_link
- joint rod_3_end_effector_joint: origin xyz=0 0 -450 -> xyz=0 0 -400; parent rod_3_link -> rod_3a_link
